Commit message: Update rx200_kinect.urdf.xacro

File: urdf/rx200_kinect.urdf.xacro (robot description, xacro)
@@ -12,13 +12,13 @@
     https://wiki.ros.org/xacro
     -->
-    <!--Kinect v2-->
-    <xacro:include filename="$(find common_sensors)/urdf/sensors/kinect2.urdf.xacro"/>
-    <xacro:kinect2 name="kinect2" parent="world">
-        <origin rpy="0 0.3 3.15" xyz="1.4 -0.08 0.2"/>
+<!--     <!--Kinect v2-->-->
+<!--     <xacro:include filename="$(find common_sensors)/urdf/sensors/kinect2.urdf.xacro"/>-->
+<!--     <xacro:kinect2 name="kinect2" parent="world">-->
+<!--         <origin rpy="0 0.3 3.15" xyz="1.4 -0.08 0.2"/>-->
 <!--        <origin rpy="0 0.2 3.15" xyz="1.3 -0.08 0.2"/>-->
 <!--        <origin rpy="0 0 -1.6" xyz="0.35 0.6 0"/>-->
 <!--        <origin rpy="0 1.5 0" xyz="0 0.1 1"/>-->
 <!--        <origin rpy="0 0.5 3" xyz="1 0 0.5"/>-->
-    </xacro:kinect2>
+<!--     </xacro:kinect2>-->
 <!--    <link name="world"/>-->
 <!---->

Commit message: fixed urdf

File: urdf/rx200_kinect.urdf.xacro (robot description, xacro)
@@ -12,13 +12,13 @@
     https://wiki.ros.org/xacro
     -->
-<!--     <!--Kinect v2-->-->
-<!--     <xacro:include filename="$(find common_sensors)/urdf/sensors/kinect2.urdf.xacro"/>-->
-<!--     <xacro:kinect2 name="kinect2" parent="world">-->
-<!--         <origin rpy="0 0.3 3.15" xyz="1.4 -0.08 0.2"/>-->
+     <!--Kinect v2-->
+     <xacro:include filename="$(find common_sensors)/urdf/sensors/kinect2.urdf.xacro"/>
+     <xacro:kinect2 name="kinect2" parent="world">
+         <origin rpy="0 0.3 3.15" xyz="1.4 -0.08 0.2"/>
 <!--        <origin rpy="0 0.2 3.15" xyz="1.3 -0.08 0.2"/>-->
 <!--        <origin rpy="0 0 -1.6" xyz="0.35 0.6 0"/>-->
 <!--        <origin rpy="0 1.5 0" xyz="0 0.1 1"/>-->
 <!--        <origin rpy="0 0.5 3" xyz="1 0 0.5"/>-->
-<!--     </xacro:kinect2>-->
+     </xacro:kinect2>
 <!--    <link name="world"/>-->
 <!---->
