Commit message: updated the zed2 pose

File: urdf/rx200_zed2.urdf.xacro (robot description, xacro)
@@ -3,33 +3,15 @@
     <!-- rx200 -->
     <xacro:include filename="$(find reactorx200_description)/urdf/rx200.urdf.xacro"/>
-    <!--Kinect-->
-    <!-- position of kinect has to be changed in common_sensors/urdf/sensors/kinect_properties.urdf.xacro
-    <xacro:include filename="$(find common_sensors)/urdf/sensors/kinect.urdf.xacro"/>
-    <xacro:sensor_kinect parent="world"/> -->
-    <!--
-    By Jay: to mount the camera in gazebo
-    https://abedgnu.github.io/Notes-ROS/chapters/ROS/10_robot_modeling/xarco.html
-    https://wiki.ros.org/xacro
-    -->
-     <!--Kinect v2-->
-<!--     <xacro:include filename="$(find common_sensors)/urdf/sensors/kinect2.urdf.xacro"/>-->
-<!--     <xacro:kinect2 name="kinect2" parent="world">-->
-<!--         <origin rpy="0 0.3 3.15" xyz="1.4 -0.08 0.2"/>-->
-<!--&lt;!&ndash;        <origin rpy="0 0.2 3.15" xyz="1.3 -0.08 0.2"/>&ndash;&gt;-->
-<!--&lt;!&ndash;        <origin rpy="0 0 -1.6" xyz="0.35 0.6 0"/>&ndash;&gt;-->
-<!--&lt;!&ndash;        <origin rpy="0 1.5 0" xyz="0 0.1 1"/>&ndash;&gt;-->
-<!--&lt;!&ndash;        <origin rpy="0 0.5 3" xyz="1 0 0.5"/>&ndash;&gt;-->
-<!--     </xacro:kinect2>-->
     <!--ZED2-->
     <xacro:include filename="$(find common_sensors)/urdf/sensors/zed2.xacro"/>
     <xacro:zed2 link_prefix="" joint_prefix="" />
     <!-- Include the Gazebo plugins for the ZED2 -->
-    <xacro:zed2_gazebo robot_ns=""/>
-<!--    <link name="world"/>-->
-<!---->
-<!--    <joint name="world_joint" type="fixed">-->
-<!--        <parent link="world"/>-->
-<!--        <child link="base_link"/>-->
-<!--        <origin xyz="0.0 0.0 1.0" rpy="0.0 0.0 0.0"/>-->
-<!--    </joint>-->
+    <xacro:zed2_gazebo robot_ns=""/>>
+    <!-- Attach the ZED2 camera to a suitable link in your robot -->
+    <!-- <link name="world"/>--> <!-- Only if not defined before -->
+    <joint name="zed2_mount_joint" type="fixed">
+        <parent link="world"/> <!-- Change to the appropriate parent link in your robot -->
+        <child link="zed2_camera_center"/>
+        <origin xyz="0.8 0 0.025" rpy="0 -0.2 ${pi}"/> <!-- Adjust the position and orientation as needed -->
+    </joint>
 </robot>

Commit message: increased the z

File: urdf/rx200_zed2.urdf.xacro (robot description, xacro)
@@ -13,5 +13,5 @@
         <parent link="world"/> <!-- Change to the appropriate parent link in your robot -->
         <child link="zed2_camera_center"/>
-        <origin xyz="0.8 0 0.025" rpy="0 -0.2 ${pi}"/> <!-- Adjust the position and orientation as needed -->
+        <origin xyz="0.8 0 0.08" rpy="0 -0.2 ${pi}"/> <!-- Adjust the position and orientation as needed -->
     </joint>
 </robot>
